File: variant-1/2x5toCortexAdapt.sch (KiCad schematic (older format))
At the start: 2 parts, among them J1 2X5_HDR, J2 ARM_10PIN

Commit message: update 3d render for variant-1
Parts:
- J1: footprint kicadlib:ARM_10_PIN_0.1_TH_RIGHTANGLE -> Connector_IDC:IDC-Header_2x05_P2.54mm_Horizontal; symbol 2X5_HDR -> kicadlib:2X5_HDR
- J2: footprint kicadlib:ARM_10_PIN -> Connector_PinSocket_1.27mm:PinSocket_2x05_P1.27mm_Vertical; symbol ARM_10PIN -> kicadlib:ARM_10PIN
Changed lines of the file:
@@
-EESchema Schematic File Version 2
-LIBS:power
-LIBS:device
-LIBS:transistors
-LIBS:conn
-LIBS:linear
-LIBS:regul
-LIBS:74xx
-LIBS:cmos4000
-LIBS:adc-dac
-LIBS:memory
-LIBS:xilinx
-LIBS:microcontrollers
-LIBS:dsp
-LIBS:microchip
-LIBS:analog_switches
-LIBS:motorola
-LIBS:texas
-LIBS:intel
-LIBS:audio
-LIBS:interface
-LIBS:digital-audio
-LIBS:philips
-LIBS:display
-LIBS:cypress
-LIBS:siliconi
-LIBS:opto
-LIBS:atmel
-LIBS:contrib
-LIBS:valves
-LIBS:kicadlib
-LIBS:2x5toCortexAdapt-cache
-EELAYER 25 0
+EESchema Schematic File Version 4
+EELAYER 30 0
 EELAYER END
 $Descr A4 11693 8268
@@
 $EndDescr
 $Comp
-L ARM_10PIN J2
+L kicadlib:ARM_10PIN J2
 U 1 1 5643BF5B
 P 5500 2400
 F 0 "J2" H 5500 1400 60  0000 C CNN
 F 1 "ARM_10PIN" H 5500 3050 60  0000 C CNN
-F 2 "kicadlib:ARM_10_PIN" H 5500 2400 60  0001 C CNN
+F 2 "Connector_PinSocket_1.27mm:PinSocket_2x05_P1.27mm_Vertical" H 5500 2400 60  0001 C CNN
 F 3 "" H 5500 2400 60  0000 C CNN
 	1    5500 2400
@@
 GND
 Wire Wire Line
-	4850 3100 5050 3100
+	4850 3100 4950 3100
 Wire Wire Line
 	5050 2500 4950 2500
 Wire Wire Line
-	4950 2200 4950 3100
+	4950 2200 4950 2500
 Connection ~ 4950 3100
 Wire Wire Line
@@
 	5000 3250 4850 3250
 $Comp
-L 2X5_HDR J1
+L kicadlib:2X5_HDR J1
 U 1 1 5643C704
 P 3000 1850
 F 0 "J1" H 3000 1350 60  0000 C CNN
 F 1 "2X5_HDR" H 3000 2250 60  0000 C CNN
-F 2 "kicadlib:ARM_10_PIN_0.1_TH_RIGHTANGLE" H 2900 1600 60  0001 C CNN
+F 2 "Connector_IDC:IDC-Header_2x05_P2.54mm_Horizontal" H 2900 1600 60  0001 C CNN
 F 3 "" H 2900 1600 60  0000 C CNN
 	1    3000 1850
 	1    0    0    -1
 $EndComp
+Wire Wire Line
+	4950 3100 5050 3100
+Wire Wire Line
+	4950 2500 4950 3100
 $EndSCHEMATC
