File: variant-1/2x5toCortexAdapt.kicad_pcb (KiCad board)
At the start: 2 copper layers, 15 x 14.2 mm, 2 parts, among them J1 2X5_HDR, J2 ARM_10PIN

Commit message: variant-1 v2 update
Routing:
- net /GND: track 14.5 -> 7.07 mm
- net /SWIM: track 13.5 -> 14.9 mm
- net /RST: track 16.5 -> 15.4 mm
- net /SWCLK: track 16.7 -> 15.9 mm, vias 1 -> 0
- removed copper zone on B.Cu, net /GND
Other:
- rule pad_to_mask_clearance: 0.2 -> 0
- board text added: "VARIANT-1"
- board text added: "github.com/noahp/ 2x5toCortexAdapt/ variant-1 v2"
- board text removed: "github.com/noahp/ 2x5toCortexAdapt v1"
Changed lines of the file:
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@@
   (general
     (thickness 1.6)
-    (drawings 9)
-    (tracks 36)
+    (drawings 10)
+    (tracks 28)
     (zones 0)
     (modules 2)
@@
   )
   (setup
-    (last_trace_width 0.25)
+    (last_trace_width 0.35)
     (user_trace_width 0.35)
     (trace_clearance 0.2)
-    (zone_clearance 0.508)
+    (zone_clearance 0.35)
     (zone_45_only no)
     (trace_min 0.2)
@@
     (pad_size 1.524 1.524)
     (pad_drill 0.762)
-    (pad_to_mask_clearance 0.2)
+    (pad_to_mask_clearance 0)
     (aux_axis_origin 0 0)
     (visible_elements FFFFFF7F)
     (pcbplotparams
-      (layerselection 0x010f0_80000001)
+      (layerselection 0x010f0_ffffffff)
       (usegerberextensions false)
       (usegerberattributes true)
@@
       (effects (font (size 0.75 0.75) (thickness 0.12)))
     )
+    (fp_line (start -2.6 -6.4) (end 2.6 -6.4) (layer F.SilkS) (width 0.15))
+    (fp_line (start -2.6 6.4) (end -2.6 -6.4) (layer F.SilkS) (width 0.15))
+    (fp_line (start 2.6 6.4) (end -2.6 6.4) (layer F.SilkS) (width 0.15))
     (fp_line (start 2.6 -6.4) (end 2.6 6.4) (layer F.SilkS) (width 0.15))
-    (fp_line (start 2.6 6.4) (end -2.6 6.4) (layer F.SilkS) (width 0.15))
-    (fp_line (start -2.6 6.4) (end -2.6 -6.4) (layer F.SilkS) (width 0.15))
-    (fp_line (start -2.6 -6.4) (end 2.6 -6.4) (layer F.SilkS) (width 0.15))
     (fp_text user 1 (at -1.535 -2.5) (layer F.SilkS)
       (effects (font (size 0.75 0.75) (thickness 0.12)))
@@
     )
   )
-  (gr_text "github.com/noahp/\n2x5toCortexAdapt\nv1" (at 155.702 114.9985 180) (layer B.Mask)
+  (gr_text VARIANT-1 (at 155.956 104.775) (layer B.SilkS)
+    (effects (font (size 1 1) (thickness 0.15)) (justify mirror))
+  )
+  (gr_text "github.com/noahp/\n2x5toCortexAdapt/\nvariant-1 v2" (at 155.702 114.9985) (layer B.Mask)
     (effects (font (size 0.5 0.5) (thickness 0.125)) (justify mirror))
   )
@@
   (gr_arc (start 158.75 105.156) (end 158.75 103.124) (angle 90) (layer Edge.Cuts) (width 0.15))
   (gr_arc (start 147.828 105.156) (end 145.796 105.156) (angle 90) (layer Edge.Cuts) (width 0.15))
-  (segment (start 150.368 105.156) (end 151.593 105.156) (width 0.35) (layer F.Cu) (net 1))
-  (segment (start 151.593 105.156) (end 151.760001 104.988999) (width 0.35) (layer F.Cu) (net 1))
-  (segment (start 151.760001 104.988999) (end 157.670766 104.988999) (width 0.35) (layer F.Cu) (net 1))
-  (segment (start 157.670766 104.988999) (end 159.540011 106.858243) (width 0.35) (layer F.Cu) (net 1))
-  (segment (start 159.540011 106.858243) (end 159.540011 111.350989) (width 0.35) (layer F.Cu) (net 1))
-  (segment (start 159.540011 111.350989) (end 158.614999 112.276001) (width 0.35) (layer F.Cu) (net 1))
-  (segment (start 158.614999 112.276001) (end 158.115 112.776) (width 0.35) (layer F.Cu) (net 1))
-  (segment (start 158.115 107.696) (end 158.115 106.988894) (width 0.35) (layer F.Cu) (net 2))
-  (segment (start 158.115 106.988894) (end 157.532107 106.406001) (width 0.35) (layer F.Cu) (net 2))
-  (segment (start 157.532107 106.406001) (end 149.078001 106.406001) (width 0.35) (layer F.Cu) (net 2))
-  (segment (start 149.078001 106.406001) (end 148.702999 106.030999) (width 0.35) (layer F.Cu) (net 2))
-  (segment (start 148.702999 106.030999) (end 147.828 105.156) (width 0.35) (layer F.Cu) (net 2))
-  (segment (start 156.845 110.236) (end 152.908 110.236) (width 0.35) (layer F.Cu) (net 3))
-  (segment (start 152.908 110.236) (end 150.368 107.696) (width 0.35) (layer F.Cu) (net 3))
-  (segment (start 156.845 108.966) (end 151.638 108.966) (width 0.35) (layer F.Cu) (net 3))
-  (segment (start 151.638 108.966) (end 150.368 107.696) (width 0.35) (layer F.Cu) (net 3))
-  (segment (start 158.115 110.236) (end 158.990001 109.360999) (width 0.35) (layer B.Cu) (net 4))
-  (segment (start 158.990001 109.360999) (end 158.990001 107.275999) (width 0.35) (layer B.Cu) (net 4))
-  (segment (start 158.990001 107.275999) (end 158.535001 106.820999) (width 0.35) (layer B.Cu) (net 4))
-  (segment (start 158.535001 106.820999) (end 155.020437 106.820999) (width 0.35) (layer B.Cu) (net 4))
-  (segment (start 155.020437 106.820999) (end 151.605436 110.236) (width 0.35) (layer B.Cu) (net 4))
-  (segment (start 151.605436 110.236) (end 150.368 110.236) (width 0.35) (layer B.Cu) (net 4))
-  (segment (start 152.908 105.664) (end 152.608001 105.963999) (width 0.35) (layer B.Cu) (net 5))
-  (segment (start 152.608001 105.963999) (end 152.608001 107.345999) (width 0.35) (layer B.Cu) (net 5))
-  (segment (start 152.608001 107.345999) (end 150.968001 108.985999) (width 0.35) (layer B.Cu) (net 5))
-  (segment (start 150.968001 108.985999) (end 149.078001 108.985999) (width 0.35) (layer B.Cu) (net 5))
-  (segment (start 149.078001 108.985999) (end 148.702999 109.361001) (width 0.35) (layer B.Cu) (net 5))
-  (segment (start 148.702999 109.361001) (end 147.828 110.236) (width 0.35) (layer B.Cu) (net 5))
-  (segment (start 158.115 108.966) (end 158.990001 108.090999) (width 0.35) (layer F.Cu) (net 5))
-  (segment (start 158.990001 108.090999) (end 158.990001 107.086064) (width 0.35) (layer F.Cu) (net 5))
-  (segment (start 158.990001 107.086064) (end 157.567937 105.664) (width 0.35) (layer F.Cu) (net 5))
-  (segment (start 157.567937 105.664) (end 152.908 105.664) (width 0.35) (layer F.Cu) (net 5))
-  (via (at 152.908 105.664) (size 0.6) (drill 0.4) (layers F.Cu B.Cu) (net 5))
+  (segment (start 158.990001 111.900999) (end 158.115 112.776) (width 0.35) (layer F.Cu) (net 1))
+  (segment (start 158.990001 107.275999) (end 158.990001 111.900999) (width 0.35) (layer F.Cu) (net 1))
+  (segment (start 156.870002 105.156) (end 158.990001 107.275999) (width 0.35) (layer F.Cu) (net 1))
+  (segment (start 150.368 105.156) (end 156.870002 105.156) (width 0.35) (layer F.Cu) (net 1))
+  (segment (start 157.230003 106.406001) (end 158.115 107.290998) (width 0.35) (layer F.Cu) (net 2))
+  (segment (start 149.078001 106.406001) (end 157.230003 106.406001) (width 0.35) (layer F.Cu) (net 2))
+  (segment (start 158.115 107.290998) (end 158.115 107.696) (width 0.35) (layer F.Cu) (net 2))
+  (segment (start 147.828 105.156) (end 149.078001 106.406001) (width 0.35) (layer F.Cu) (net 2))
+  (segment (start 147.828 107.696) (end 150.368 107.696) (width 0.35) (layer B.Cu) (net 3))
+  (segment (start 156.845 108.966) (end 156.845 110.236) (width 0.35) (layer F.Cu) (net 3))
+  (segment (start 155.969999 111.900999) (end 156.845 112.776) (width 0.35) (layer F.Cu) (net 3))
+  (segment (start 155.969999 111.111001) (end 155.969999 111.900999) (width 0.35) (layer F.Cu) (net 3))
+  (segment (start 156.845 110.236) (end 155.969999 111.111001) (width 0.35) (layer F.Cu) (net 3))
+  (segment (start 159.540011 108.810989) (end 158.115 110.236) (width 0.35) (layer B.Cu) (net 4))
+  (segment (start 159.540011 107.048178) (end 159.540011 108.810989) (width 0.35) (layer B.Cu) (net 4))
+  (segment (start 158.762822 106.270989) (end 159.540011 107.048178) (width 0.35) (layer B.Cu) (net 4))
+  (segment (start 154.333011 106.270989) (end 158.762822 106.270989) (width 0.35) (layer B.Cu) (net 4))
+  (segment (start 150.368 110.236) (end 154.333011 106.270989) (width 0.35) (layer B.Cu) (net 4))
+  (segment (start 158.990001 107.275999) (end 158.990001 108.090999) (width 0.35) (layer B.Cu) (net 5))
+  (segment (start 158.535001 106.820999) (end 158.990001 107.275999) (width 0.35) (layer B.Cu) (net 5))
+  (segment (start 156.044999 106.820999) (end 158.535001 106.820999) (width 0.35) (layer B.Cu) (net 5))
+  (segment (start 158.990001 108.090999) (end 158.115 108.966) (width 0.35) (layer B.Cu) (net 5))
+  (segment (start 151.379997 111.486001) (end 156.044999 106.820999) (width 0.35) (layer B.Cu) (net 5))
+  (segment (start 149.078001 111.486001) (end 151.379997 111.486001) (width 0.35) (layer B.Cu) (net 5))
+  (segment (start 147.828 110.236) (end 149.078001 111.486001) (width 0.35) (layer B.Cu) (net 5))
+  (segment (start 147.828 112.776) (end 150.368 112.776) (width 0.35) (layer F.Cu) (net 6))
+  (segment (start 151.765 112.776) (end 156.845 107.696) (width 0.35) (layer B.Cu) (net 6))
   (segment (start 150.368 112.776) (end 151.765 112.776) (width 0.35) (layer B.Cu) (net 6))
-  (segment (start 151.765 112.776) (end 156.845 107.696) (width 0.35) (layer B.Cu) (net 6))
-  (segment (start 147.828 112.776) (end 150.368 112.776) (width 0.35) (layer B.Cu) (net 6))
   (zone (net 3) (net_name /GND) (layer F.Cu) (hatch edge 0.508)
     (connect_pads (clearance 0.508))
@@
     )
   )
-  (zone (net 3) (net_name /GND) (layer B.Cu) (hatch edge 0.508)
-    (connect_pads (clearance 0.508))
+  (zone (net 3) (net_name /GND) (layer F.Cu) (hatch edge 0.508)
+    (connect_pads (clearance 0.35))
     (min_thickness 0.254)
-    (fill yes (arc_segments 16) (thermal_gap 0.508) (thermal_bridge_width 0.508))
+    (fill yes (arc_segments 16) (thermal_gap 0.35) (thermal_bridge_width 0.35))
     (polygon
       (pts
