File: variant-x/2x5toCortexAdapt.kicad_pcb (KiCad board)
At the start: 2 copper layers, 25.4 x 15 mm, 5 parts, among them J1 Conn_01x04, J2 Conn_01x04, J3 2X5_HDR, J4 Conn_01x04, J5 ARM_10PIN

Commit message: save
Parts:
- J1, J2, J4: footprint Connector_PinHeader_2.54mm:PinHeader_1x04_P2.54mm_Vertical -> project-lib:PinHeader_1x04_P2.54mm_Vertical
- J3: footprint kicadlib:ARM_10_PIN_0.1_TH_RIGHTANGLE -> project-lib:IDC-Header_2x05_P2.54mm_Horizontal
- moved J3 24.5 mm to (115.4, 104.0)
Routing:
- net /GND: track 3.81 -> 1.27 mm
- net /3.3V: track 2.54 -> 0.00 mm
